File: LV3-Dash.kicad_pcb (KiCad board)
At the start: 2 copper layers, 90 x 50 mm, 93 parts, among them J1 USB_C_Receptacle_USB2.0_16P, J2 FTSH-105-01-L-DV-K-A, J3 Conn_01x04_MountingPin, J4 Conn_01x05_Pin, J5 Conn_01x05_MountingPin, J6 MSD-11-A, J7 62684-401100AHLF, U1 STM32H743VITx, U2 TJA1051T-3, U4 LMR51625YDDCR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

Commit message: r1 final (see changelog.md)
Parts:
- added J8: Conn_01x03_Pin, Connector_PinHeader_2.54mm:PinHeader_1x03_P2.54mm_Vertical, F.Cu at (53.0, 58.9)
- added R29: 5.1k, Resistor_SMD:R_0603_1608Metric_Pad0.98x0.95mm_HandSolder, B.Cu at (62.2, 83.3)
- J4: value Conn_01x05_Pin -> Conn_01x08_Pin; footprint Connector_PinHeader_2.54mm:PinHeader_1x05_P2.54mm_Vertical -> Connector_PinHeader_2.54mm:PinHeader_1x08_P2.54mm_Vertical
- moved R5 1.15 mm to (110.0, 55.1)
- moved *R23 0.87 mm to (63.8, 83.3), turned to 90 degrees
- renumbered R23 to *R23
Connections:
- U1 pad 3: unconnected-(U1-PE4-Pad3) -> SAI_FS
- U1 pad 4: unconnected-(U1-PE5-Pad4) -> SAI_SCK
- U1 pad 5: unconnected-(U1-PE6-Pad5) -> SAI_SD
Routing:
- net GND: track 653.5 -> 696.8 mm
- net CTP_SDA: track 16.2 -> 51.0 mm, vias 0 -> 4
- net CTP_SCL: track 17.7 -> 51.0 mm, vias 0 -> 4
- net SAI_FS: track 0.00 -> 23.0 mm, vias 0 -> 2
- net SAI_SCK: track 0.00 -> 22.5 mm, vias 0 -> 2
- net SAI_SD: track 0.00 -> 22.2 mm, vias 0 -> 2
- net BOOT0: track 95.5 -> 99.0 mm, vias 3 -> 5
- net Net-(D2-A): track 93.7 -> 91.7 mm
- net SD_EN: track 18.6 -> 16.7 mm
- net LCD_R6: track 35.9 -> 37.2 mm
- net BKLT_CTRL: track 50.2 -> 51.4 mm
- net CTP_INT: track 16.8 -> 17.8 mm
- net LCD_HSYNC: track 18.8 -> 19.8 mm
- net CTP_RST: track 16.3 -> 17.2 mm
- net LCD_R5: track 49.3 -> 50.2 mm
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Other:
- board text added: "(shared with touch panel)"
- board text added: "D12•SCL"
- board text added: "D13•SDA"
- board text added: "E4•FS"
- board text added: "E5•BCLK"
- board text added: "E6•SD"
- board text added: "I2C"
- board text added: "SAI"
- board text added: "r1 • Mar 2026 Cy Westbrook"
- board text added: "r1 • Mar 2026 • Cy Westbrook"
- board text removed: "r0 • Jan 2026 Cy Westbrook"
- board text removed: "r0 • Jan 2026 • Cy Westbrook"
